File: hardware/_saved_audio-controlled-neopixel.sch (KiCad schematic (older format))
At the start: 61 parts, among them J1 Phoenix MPT, J2 KF2EDGK, J3 KF2EDGK, J4 KF2EDGK, J5 Conn_01x01_Female, J6 Conn_01x01_Female, J7 Conn_01x01_Female, J8 Conn_01x01_Female, SW1 SW_SPST, U1 LM324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

Commit message: update schematic to use 3.5mm audio I/O
Parts:
- removed J1: Phoenix MPT, TerminalBlock_Phoenix:TerminalBlock_Phoenix_MPT-0,5-6-2.54_1x06_P2.54mm_Horizontal, symbol Connector:Conn_01x06_Female
- added J1, J2: AudioJack3_Ground, Footprints:Jack_3.5mm_PJ320E_Horizontal, symbol Connector:AudioJack3_Ground
- renumbered J2 to J3, J3 to J4, J4 to J5, J5 to J7, J7 to J8, J8 to J9
Connections:
- wire segments 245 -> 238
Other:
- moved on the sheet: C19, D10, F1, J3, J4, J5, J6, J7, J9
