File: hardware/audio-controlled-neopixel.sch (KiCad schematic (older format))
At the start: 63 parts, among them J1 Phoenix MPT, J2 Conn_01x01_Female, J3 Phoenix MPT 3, J4 Phoenix MKDS 2, J5 Conn_01x01_Female, J6 Conn_01x01_Female, J7 Conn_01x01_Female, SW1 SW_SPST, U1 NE5532, U2 NE5532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

Commit message: Tweaked filter values for treble in schematic, added gamma correction for LEDs.
Parts:
- removed U4: TMA0512D, Footprints:TMAxxxxD, symbol custom:TMAxxxxD
- R10, R12: value 4K7 -> 7K5
Connections:
- wire segments 237 -> 235

Commit message: Updated schematic and PCB to use SMD components for ease of manufacture.
Parts:
- removed C17, C18: 100n, Capacitor_THT:C_Disc_D4.3mm_W1.9mm_P5.00mm, symbol Device:C_Small
- removed U3: NE5532, Package_DIP:DIP-8_W7.62mm_LongPads, symbol Amplifier_Operational:NE5532
- added C21, C22: 100n, Capacitor_SMD:C_0805_2012Metric, symbol Device:C_Small
- added U3: LM324, Package_SO:SOIC-14_3.9x8.7mm_P1.27mm, symbol Amplifier_Operational:LM324
- added U4: TMA0512D, Footprints:TMAxxxxD, symbol custom:TMAxxxxD
- C1, C2: footprint Capacitor_THT:CP_Radial_D5.0mm_P2.00mm -> Capacitor_SMD:C_0805_2012Metric
- C10, C11, C12, C13, C14, C15, C16, C20, C3, C4, C5, C6, C7, C8, C9: footprint Capacitor_THT:C_Disc_D4.3mm_W1.9mm_P5.00mm -> Capacitor_SMD:C_0805_2012Metric
- D1, D4, D5, D6: footprint Diode_THT:D_DO-35_SOD27_P7.62mm_Horizontal -> Diode_SMD:D_SOD-123
- D10, D3, D7, D8, D9: value BAT85 -> 1N5819; footprint Diode_THT:D_DO-35_SOD27_P7.62mm_Horizontal -> Diode_SMD:D_SOD-123
- D2: footprint LED_THT:LED_D3.0mm_Horizontal_O1.27mm_Z2.0mm -> LED_SMD:LED_0805_2012Metric
- F1: value 611-9302 -> 176-9047
- J3: value Phoenix MPT 3 -> KF2EDGK; footprint TerminalBlock_Phoenix:TerminalBlock_Phoenix_MPT-0,5-3-2.54_1x03_P2.54mm_Horizontal -> Connector_Phoenix_MSTB:PhoenixContact_MSTBA_2,5_3-G-5,08_1x03_P5.08mm_Horizontal
- J4: value Phoenix MKDS 2 -> KF2EDGK; footprint TerminalBlock_Phoenix:TerminalBlock_Phoenix_PT-1,5-2-3.5-H_1x02_P3.50mm_Horizontal -> Connector_Phoenix_MSTB:PhoenixContact_MSTBA_2,5_2-G_1x02_P5.00mm_Horizontal
- R1, R10, R11, R12, R13, R14, R15, R16, R17, R18, R2, R3, R4, R6, R7, R8, R9: footprint Resistor_THT:R_Axial_DIN0204_L3.6mm_D1.6mm_P7.62mm_Horizontal -> Resistor_SMD:R_0805_2012Metric
- R5: value 100K -> 200K; footprint Resistor_THT:R_Axial_DIN0204_L3.6mm_D1.6mm_P2.54mm_Vertical -> Resistor_SMD:R_0805_2012Metric
- U1: value NE5532 -> LM358; footprint Package_DIP:DIP-8_W7.62mm_LongPads -> Package_SO:SOIC-8_3.9x4.9mm_P1.27mm
- U2: footprint Package_DIP:DIP-8_W7.62mm_LongPads -> Package_SO:SOIC-8_3.9x4.9mm_P1.27mm
Connections:
- wire segments 235 -> 247
Other:
- note added: "2.5KHz-20KHz"
- note added: "413Hz-2.5KHz"
- note removed: "3.4KHz-20KHz"
- note removed: "413Hz-3.4KHz"
- moved on the sheet: A1, C1, C10, C11, C12, C13, C14, C15, C16, C2, C20, C3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

Commit message: Added pdf schematic
Parts:
- U4: symbol custom:TMAxxxxD -> audio-controlled-neopixel-rescue:TMAxxxxD-custom
Changed lines of the file:
@@
 $EndComp
 $Comp
-L custom:TMAxxxxD U4
+L audio-controlled-neopixel-rescue:TMAxxxxD-custom U4
 U 1 1 5BF146EE
 P 3750 1100

Commit message: updated schematic to reduce component count, PCB update to match
Parts:
- removed C1, C2: 10u, Capacitor_SMD:C_0805_2012Metric, symbol Device:C_Small
- removed C21, C22: 100n, Capacitor_SMD:C_0805_2012Metric, symbol Device:C_Small
- removed J2: Conn_01x01_Female, MountingHole:MountingHole_3.2mm_M3, symbol Connector:Conn_01x01_Female
- removed U1: LM358, Package_SO:SOIC-8_3.9x4.9mm_P1.27mm, symbol Amplifier_Operational:NE5532
- removed U2: NE5532, Package_SO:SOIC-8_3.9x4.9mm_P1.27mm, symbol Amplifier_Operational:NE5532
- added C1, C2: 10u, Capacitor_THT:CP_Radial_D5.0mm_P2.00mm, symbol Device:CP_Small
- added J2: KF2EDGK, TerminalBlock_Phoenix:TerminalBlock_Phoenix_MPT-0,5-3-2.54_1x03_P2.54mm_Horizontal, symbol Connector:Conn_01x03_Female
- added J8: Conn_01x01_Female, MountingHole:MountingHole_3.2mm_M3, symbol Connector:Conn_01x01_Female
- added U1: LM324, Package_SO:SOIC-14_3.9x8.7mm_P1.27mm, symbol Amplifier_Operational:LM324
- C10, C11, C12, C3: value 1u -> 100n
- C19: value EEUFM1C102 -> 330u 35V
- R14, R15, R16: value 100K -> 1M
- RV1: value 10K -> 10KA
- U4: symbol audio-controlled-neopixel-rescue:TMAxxxxD-custom -> custom:TMAxxxxD
Connections:
- net labels added: High, Low, Mid
- net labels removed: High_out, Low_out, Mid_out, Passthru_L, Passthru_R
- wire segments 247 -> 245
Other:
- moved on the sheet: C15, C16, C19, J3, R2, R3, R4, R5, RV1A, RV1B, U3E

Commit message: update schematic to use 3.5mm audio I/O
Parts:
- removed J1: Phoenix MPT, TerminalBlock_Phoenix:TerminalBlock_Phoenix_MPT-0,5-6-2.54_1x06_P2.54mm_Horizontal, symbol Connector:Conn_01x06_Female
- added J1, J2: AudioJack3_Ground, Footprints:Jack_3.5mm_PJ320E_Horizontal, symbol Connector:AudioJack3_Ground
- renumbered J2 to J3, J3 to J4, J4 to J5, J5 to J7, J7 to J8, J8 to J9
Connections:
- wire segments 245 -> 238
Other:
- moved on the sheet: C19, D10, F1, J3, J4, J5, J6, J7, J9

Commit message: clean up schematic and PCB
Parts:
- removed C16: 100n, Capacitor_SMD:C_0805_2012Metric, symbol Device:C_Small
Connections:
- wire segments 238 -> 235
Other:
- moved on the sheet: A1, C13, C14, C15, C19, C20, C3, D1, D10, D2, D3, F1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

Commit message: add attenuator for peak level calibration
Parts:
- added R19: 10K, Resistor_SMD:R_0805_2012Metric, symbol Device:R_Small
- added R20: 100K, Resistor_SMD:R_0805_2012Metric, symbol Device:R_Small
- U4: symbol custom:TMAxxxxD -> audio-controlled-neopixel-rescue:TMAxxxxD-custom
Connections:
- wire segments 235 -> 241
Other:
- note added: "R19/20 define attenuation for peak level calibration"
Changed lines of the file:
@@
 EESchema Schematic File Version 4
-LIBS:audio-controlled-neopixel-cache
 EELAYER 26 0
 EELAYER END
@@
 Wire Wire Line
 	8525 1775 8525 1725
-Text Label 5200 4550 2    50   ~ 0
+Text Label 4950 4550 2    50   ~ 0
 Buf_input
 $Comp
@@
 	5575 4550 5925 4550
 Wire Wire Line
-	5575 4850 5575 4800
+	5575 4850 5575 4825
 $Comp
 L Device:C_Small C3
@@
 $EndComp
 Wire Wire Line
-	5200 4550 5275 4550
+	5200 4550 5250 4550
 Wire Wire Line
 	2525 3375 2525 3500
@@
 $EndComp
 $Comp
-L custom:TMAxxxxD U4
+L audio-controlled-neopixel-rescue:TMAxxxxD-custom U4
 U 1 1 5BF146EE
 P 3150 2175
@@
 Wire Wire Line
 	1625 7125 1625 7325
+$Comp
+L Device:R_Small R19
+U 1 1 5C3F66FF
+P 5100 4550
+F 0 "R19" H 5175 4575 50  0000 L CNN
+F 1 "10K" H 5175 4500 50  0000 L CNN
+F 2 "Resistor_SMD:R_0805_2012Metric" H 5100 4550 50  0001 C CNN
+F 3 "~" H 5100 4550 50  0001 C CNN
+	1    5100 4550
+	0    -1   -1   0
+$EndComp
+$Comp
+L Device:R_Small R20
+U 1 1 5C3F6822
+P 5250 4700
+F 0 "R20" H 5325 4725 50  0000 L CNN
+F 1 "100K" H 5325 4650 50  0000 L CNN
+F 2 "Resistor_SMD:R_0805_2012Metric" H 5250 4700 50  0001 C CNN
+F 3 "~" H 5250 4700 50  0001 C CNN
+	1    5250 4700
+	-1   0    0    1
+$EndComp
+Wire Wire Line
+	5250 4600 5250 4550
+Connection ~ 5250 4550
+Wire Wire Line
+	5250 4550 5275 4550
+Wire Wire Line
+	5250 4800 5250 4825
+Wire Wire Line
+	5250 4825 5575 4825
+Connection ~ 5575 4825
+Wire Wire Line
+	5575 4825 5575 4800
+Wire Wire Line
+	4950 4550 5000 4550
+Text Notes 3325 4975 0    50   ~ 0
+R19/20 define attenuation for peak level calibration
 $EndSCHEMATC

Commit message: updated some footprints and symbols
Parts:
- removed J1, J2: AudioJack3_Ground, Footprints:Jack_3.5mm_PJ320E_Horizontal, symbol Connector:AudioJack3_Ground
- removed U4: TMA0512D, Footprints:TMAxxxxD, symbol audio-controlled-neopixel-rescue:TMAxxxxD-custom
- added J1, J2: AudioJack4, Connector_Audio:Jack_3.5mm_PJ320D_Horizontal, symbol Connector:AudioJack4
- added U2: TMA0512D, custom:TMA-0512D, symbol TMA_2412D:TMA_2412D
Changed lines of the file:
@@
 Input_R
 Wire Wire Line
-	2650 2075 2575 2075
-Wire Wire Line
-	2575 2075 2575 2125
-Wire Wire Line
-	2650 1975 2575 1975
-Wire Wire Line
-	2575 1975 2575 1925
+	2550 2000 2475 2000
+Wire Wire Line
+	2475 2000 2475 2050
+Wire Wire Line
+	2550 1900 2475 1900
+Wire Wire Line
+	2475 1900 2475 1850
 $Comp
 L power:+12V #PWR0106
 U 1 1 5BF24254
-P 3675 1900
-F 0 "#PWR0106" H 3675 1750 50  0001 C CNN
-F 1 "+12V" H 3690 2073 50  0000 C CNN
-F 2 "" H 3675 1900 50  0001 C CNN
-F 3 "" H 3675 1900 50  0001 C CNN
-	1    3675 1900
+P 4075 1875
+F 0 "#PWR0106" H 4075 1725 50  0001 C CNN
+F 1 "+12V" H 4090 2048 50  0000 C CNN
+F 2 "" H 4075 1875 50  0001 C CNN
+F 3 "" H 4075 1875 50  0001 C CNN
+	1    4075 1875
 	1    0    0    -1
 $EndComp
@@
 L power:-12V #PWR0107
 U 1 1 5BF242D9
-P 3725 2025
-F 0 "#PWR0107" H 3725 2125 50  0001 C CNN
-F 1 "-12V" H 3740 2198 50  0000 C CNN
-F 2 "" H 3725 2025 50  0001 C CNN
-F 3 "" H 3725 2025 50  0001 C CNN
-	1    3725 2025
+P 4125 2000
+F 0 "#PWR0107" H 4125 2100 50  0001 C CNN
+F 1 "-12V" H 4140 2173 50  0000 C CNN
+F 2 "" H 4125 2000 50  0001 C CNN
+F 3 "" H 4125 2000 50  0001 C CNN
+	1    4125 2000
 	0    1    1    0
 $EndComp
 Wire Wire Line
-	3675 2150 3675 2125
-Wire Wire Line
-	3675 2125 3650 2125
-Wire Wire Line
-	3675 1900 3675 1925
-Wire Wire Line
-	3675 1925 3650 1925
-Wire Wire Line
-	3650 2025 3725 2025
+	4075 2125 4075 2100
+Wire Wire Line
+	4075 2100 4050 2100
+Wire Wire Line
+	4075 1875 4075 1900
+Wire Wire Line
+	4075 1900 4050 1900
+Wire Wire Line
+	4050 2000 4125 2000
 $Comp
 L Diode:BAT85 D3
@@
 L power:GND #PWR0111
 U 1 1 5C0E2BC2
-P 3675 2150
-F 0 "#PWR0111" H 3675 1900 50  0001 C CNN
-F 1 "GND" H 3680 1977 50  0000 C CNN
-F 2 "" H 3675 2150 50  0001 C CNN
-F 3 "" H 3675 2150 50  0001 C CNN
-	1    3675 2150
+P 4075 2125
+F 0 "#PWR0111" H 4075 1875 50  0001 C CNN
+F 1 "GND" H 4080 1952 50  0000 C CNN
+F 2 "" H 4075 2125 50  0001 C CNN
+F 3 "" H 4075 2125 50  0001 C CNN
+	1    4075 2125
 	1    0    0    -1
 $EndComp
@@
 L power:GND #PWR0112
 U 1 1 5C111DEF
-P 2575 2125
-F 0 "#PWR0112" H 2575 1875 50  0001 C CNN
-F 1 "GND" H 2580 1952 50  0000 C CNN
-F 2 "" H 2575 2125 50  0001 C CNN
-F 3 "" H 2575 2125 50  0001 C CNN
-	1    2575 2125
+P 2475 2050
+F 0 "#PWR0112" H 2475 1800 50  0001 C CNN
+F 1 "GND" H 2480 1877 50  0000 C CNN
+F 2 "" H 2475 2050 50  0001 C CNN
+F 3 "" H 2475 2050 50  0001 C CNN
+	1    2475 2050
 	1    0    0    -1
 $EndComp
@@
 L power:+5V #PWR0125
 U 1 1 5C1563B7
-P 2575 1925
-F 0 "#PWR0125" H 2575 1775 50  0001 C CNN
-F 1 "+5V" H 2590 2098 50  0000 C CNN
-F 2 "" H 2575 1925 50  0001 C CNN
-F 3 "" H 2575 1925 50  0001 C CNN
-	1    2575 1925
+P 2475 1850
+F 0 "#PWR0125" H 2475 1700 50  0001 C CNN
+F 1 "+5V" H 2490 2023 50  0000 C CNN
+F 2 "" H 2475 1850 50  0001 C CNN
+F 3 "" H 2475 1850 50  0001 C CNN
+	1    2475 1850
 	1    0    0    -1
 $EndComp
@@
 	1    0    0    -1
 $EndComp
-$Comp
-L audio-controlled-neopixel-rescue:TMAxxxxD-custom U4
-U 1 1 5BF146EE
-P 3150 2175
-F 0 "U4" H 2750 2625 50  0000 L CNN
-F 1 "TMA0512D" H 2750 2525 50  0000 L CNN
-F 2 "Footprints:TMAxxxxD" H 3250 2075 50  0001 C CIN
-F 3 "" H 3150 2175 50  0001 C CNN
-	1    3150 2175
-	1    0    0    -1
-$EndComp
+Text Label 975  3825 2    50   ~ 0
+Input_L
 Text Label 975  3175 2    50   ~ 0
-Input_L
-Text Label 975  3825 2    50   ~ 0
 Input_R
 Wire Wire Line
@@
 Wire Wire Line
 	1200 1300 1200 1200
-$Comp
-L Connector:AudioJack3_Ground J1
-U 1 1 5C505DD1
-P 775 900
-F 0 "J1" H 751 1242 50  0000 C CNN
-F 1 "AudioJack3_Ground" H 751 1151 50  0000 C CNN
-F 2 "Footprints:Jack_3.5mm_PJ320E_Horizontal" H 775 900 50  0001 C CNN
-F 3 "~" H 775 900 50  0001 C CNN
-	1    775  900
-	1    0    0    -1
-$EndComp
-Wire Wire Line
-	575  1200 1200 1200
-Connection ~ 1200 1200
-$Comp
-L Connector:AudioJack3_Ground J2
-U 1 1 5C561508
-P 1600 900
-F 0 "J2" H 1600 1225 50  0000 R CNN
-F 1 "AudioJack3_Ground" H 1850 1150 50  0000 R CNN
-F 2 "Footprints:Jack_3.5mm_PJ320E_Horizontal" H 1600 900 50  0001 C CNN
-F 3 "~" H 1600 900 50  0001 C CNN
-	1    1600 900
-	-1   0    0    -1
-$EndComp
-Wire Wire Line
-	1800 1200 1200 1200
 Wire Wire Line
 	925  7325 925  7300
@@
 Text Notes 3325 4975 0    50   ~ 0
 R19/20 define attenuation for peak level calibration
+$Comp
+L Connector:AudioJack4 J1
+U 1 1 5C4A06F4
+P 775 1100
+F 0 "J1" H 445 983 50  0000 R CNN
+F 1 "AudioJack4" H 445 1074 50  0000 R CNN
+F 2 "Connector_Audio:Jack_3.5mm_PJ320D_Horizontal" H 775 1100 50  0001 C CNN
+F 3 "~" H 775 1100 50  0001 C CNN
+	1    775  1100
+	1    0    0    1
+$EndComp
+Wire Wire Line
+	975  1200 1200 1200
+$Comp
+L Connector:AudioJack4 J2
+U 1 1 5C4A1B28
+P 1600 1100
+F 0 "J2" H 1270 983 50  0000 R CNN
+F 1 "AudioJack4" H 1270 1074 50  0000 R CNN
+F 2 "Connector_Audio:Jack_3.5mm_PJ320D_Horizontal" H 1600 1100 50  0001 C CNN
+F 3 "~" H 1600 1100 50  0001 C CNN
+	1    1600 1100
+	-1   0    0    1
+$EndComp
+Wire Wire Line
+	1400 1200 1200 1200
+Connection ~ 1200 1200
+$Comp
+L TMA_2412D:TMA_2412D U2
+U 1 1 5C4B4FE3
+P 2550 1900
+F 0 "U2" H 3300 2165 50  0000 C CNN
+F 1 "TMA0512D" H 3300 2074 50  0000 C CNN
+F 2 "custom:TMA-0512D" H 3900 2000 50  0001 L CNN
+F 3 "http://docs-emea.rs-online.com/webdocs/0e18/0900766b80e182f0.pdf" H 3900 1900 50  0001 L CNN
+F 4 "TMA2412D unregulated DC-DC,+/-12V 1W 1W Isolated DC-DC Converter, Vin 21.6" H 3900 1800 50  0001 L CNN "Description"
+F 5 "Traco Power" H 3900 1600 50  0001 L CNN "Manufacturer_Name"
+F 6 "TMA 2412D" H 3900 1500 50  0001 L CNN "Manufacturer_Part_Number"
+F 7 "1247598" H 3900 1400 50  0001 L CNN "RS Part Number"
+F 8 "http://uk.rs-online.com/web/p/products/1247598" H 3900 1300 50  0001 L CNN "RS Price/Stock"
+F 9 "495-TMA-2412D" H 3900 1200 50  0001 L CNN "Mouser Part Number"
+F 10 "https://www.mouser.com/Search/Refine.aspx?Keyword=495-TMA-2412D" H 3900 1100 50  0001 L CNN "Mouser Price/Stock"
+	1    2550 1900
+	1    0    0    -1
+$EndComp
 $EndSCHEMATC
